File: eagle/Zeitraffer_V0.1.sch (EAGLE design)
At the start: 51 parts, among them IC1 LM317MSTT3, IC2 L293D, K1 FTR-B4S, Q1 600mA/40V, Q2 310mA/60V/1.6Ω, Q3 600mA/40V, Y1 12MHz

Commit message: banana
Parts:
- added C16: (no value), resistor:C-EUC0805
Connections:
- net 3.3V: now also C16.1
- net GND: now also C16.2
Changed lines of the file:
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@@
 <part name="J3" library="SparkFun-Connectors" deviceset="USB_MICRO-B" device="_SMT"/>
 <part name="SUPPLY11" library="SparkFun-PowerSymbols" deviceset="3.3V" device=""/>
+<part name="C16" library="resistor" library_urn="urn:adsk.eagle:library:348" deviceset="C-EU" device="C0805" package3d_urn="urn:adsk.eagle:package:26137/1"/>
 </parts>
 <sheets>
@@
 <instance part="J3" gate="G$1" x="35.56" y="45.72" rot="R180"/>
 <instance part="SUPPLY11" gate="G$1" x="297.18" y="78.74"/>
+<instance part="C16" gate="G$1" x="322.58" y="55.88"/>
 </instances>
 <busses>
@@
 <wire x1="297.18" y1="48.26" x2="297.18" y2="43.18" width="0.1524" layer="91"/>
 <junction x="297.18" y="43.18"/>
+<wire x1="297.18" y1="48.26" x2="322.58" y2="48.26" width="0.1524" layer="91"/>
+<junction x="297.18" y="48.26"/>
+<pinref part="C16" gate="G$1" pin="2"/>
+<wire x1="322.58" y1="48.26" x2="322.58" y2="50.8" width="0.1524" layer="91"/>
 </segment>
 <segment>
@@
 <wire x1="297.18" y1="63.5" x2="297.18" y2="78.74" width="0.1524" layer="91"/>
 <pinref part="SUPPLY11" gate="G$1" pin="3.3V"/>
+<pinref part="C16" gate="G$1" pin="1"/>
+<wire x1="322.58" y1="58.42" x2="322.58" y2="63.5" width="0.1524" layer="91"/>
+<wire x1="322.58" y1="63.5" x2="297.18" y2="63.5" width="0.1524" layer="91"/>
+<junction x="297.18" y="63.5"/>
 </segment>
 </net>
