File: eagle/Zeitraffer_V0.1.brd (EAGLE design)
At the start: 70 x 50 mm, 51 parts, among them IC1 LM317MSTT3, IC2 L293D, K1 FTR-B4S, Q1 600mA/40V, Q2 310mA/60V/1.6Ω, Q3 600mA/40V, Y1 12MHz

Commit message: banana
Parts:
- added C16: (no value), resistor:C0805
- moved C11 0.38 mm to (13.6, 46.2)
- moved C12 0.38 mm to (5.97, 46.2)
- moved Y1 0.38 mm to (9.78, 46.2)
Connections:
- net 3.3V: now also C16.1
- net GND: now also C16.2
Routing:
- net 3.3V: track 173.3 -> 167.8 mm
- net GPIO0: track 65.0 -> 67.1 mm, vias 1 -> 3
- net DRV1: track 49.3 -> 50.8 mm
- net N$14: track 6.02 -> 6.86 mm
- net VIN: track 108.6 -> 109.3 mm
- net GND: track 13.1 -> 12.7 mm, vias 36 -> 56
Other:
- board text added: "C:/Users/Fry/Desktop/BANANA.bmp"
- board text added: "stepsie-pixie v0.1"

Commit message: final touchups generated gerber
Routing:
- net S3: track 71.7 -> 70.6 mm
- net GND: vias 56 -> 76
